File: kicad/burp_fart.kicad_sch (KiCad schematic)
At the start: 39 parts

Commit message: update: makes edges rounded
Parts:
- renumbered L_SW__0 to L_SW__00, L_SW__1 to L_SW__01, L_SW__2 to L_SW__02, L_SW__3 to L_SW__03, L_SW__4 to L_SW__04
Changed lines of the file:
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@@
   (symbol (lib_id "CherryMX:CherryMX") (at 73.66 63.5 0) (unit 1)
     (in_bom yes) (on_board yes) (fields_autoplaced)
-    (property "Reference" "L_SW__2" (id 0) (at 73.66 55.88 0))
+    (property "Reference" "L_SW__02" (id 0) (at 73.66 55.88 0))
     (property "Value" "L02 (C)" (id 1) (at 73.66 58.42 0))
     (property "Footprint" "burp_fart_keyswitches:Kailh_socket_MX_pads_flipped" (id 2) (at 73.66 62.865 0)
@@
   (symbol (lib_id "CherryMX:CherryMX") (at 119.38 63.5 0) (unit 1)
     (in_bom yes) (on_board yes) (fields_autoplaced)
-    (property "Reference" "L_SW__4" (id 0) (at 119.38 55.88 0))
+    (property "Reference" "L_SW__04" (id 0) (at 119.38 55.88 0))
     (property "Value" "L04 (B)" (id 1) (at 119.38 58.42 0))
     (property "Footprint" "burp_fart_keyswitches:Kailh_socket_MX_pads_flipped" (id 2) (at 119.38 62.865 0)
@@
   (symbol (lib_id "CherryMX:CherryMX") (at 96.52 63.5 0) (unit 1)
     (in_bom yes) (on_board yes) (fields_autoplaced)
-    (property "Reference" "L_SW__3" (id 0) (at 96.52 55.88 0))
+    (property "Reference" "L_SW__03" (id 0) (at 96.52 55.88 0))
     (property "Value" "L03 (V)" (id 1) (at 96.52 58.42 0))
     (property "Footprint" "burp_fart_keyswitches:Kailh_socket_MX_pads_flipped" (id 2) (at 96.52 62.865 0)
@@
   (symbol (lib_id "CherryMX:CherryMX") (at 50.8 63.5 0) (unit 1)
     (in_bom yes) (on_board yes) (fields_autoplaced)
-    (property "Reference" "L_SW__1" (id 0) (at 50.8 55.88 0))
+    (property "Reference" "L_SW__01" (id 0) (at 50.8 55.88 0))
     (property "Value" "L01 (X)" (id 1) (at 50.8 58.42 0))
     (property "Footprint" "burp_fart_keyswitches:Kailh_socket_MX_pads_flipped" (id 2) (at 50.8 62.865 0)
@@
   (symbol (lib_id "CherryMX:CherryMX") (at 27.94 63.5 0) (unit 1)
     (in_bom yes) (on_board yes) (fields_autoplaced)
-    (property "Reference" "L_SW__0" (id 0) (at 27.94 55.88 0))
+    (property "Reference" "L_SW__00" (id 0) (at 27.94 55.88 0))
     (property "Value" "L00 (Z)" (id 1) (at 27.94 58.42 0))
     (property "Footprint" "burp_fart_keyswitches:Kailh_socket_MX_pads_flipped" (id 2) (at 27.94 62.865 0)
@@
     )
     (path "/a4253283-4522-4851-b262-618a1cd59c2b"
-      (reference "L_SW__0") (unit 1) (value "L00 (Z)") (footprint "burp_fart_keyswitches:Kailh_socket_MX_pads_flipped")
+      (reference "L_SW__00") (unit 1) (value "L00 (Z)") (footprint "burp_fart_keyswitches:Kailh_socket_MX_pads_flipped")
     )
     (path "/a2904351-a845-4b6b-968f-bb69dbdfee76"
-      (reference "L_SW__1") (unit 1) (value "L01 (X)") (footprint "burp_fart_keyswitches:Kailh_socket_MX_pads_flipped")
+      (reference "L_SW__01") (unit 1) (value "L01 (X)") (footprint "burp_fart_keyswitches:Kailh_socket_MX_pads_flipped")
     )
     (path "/060fd6c1-c0c3-4731-93d4-83c931a4e349"
-      (reference "L_SW__2") (unit 1) (value "L02 (C)") (footprint "burp_fart_keyswitches:Kailh_socket_MX_pads_flipped")
+      (reference "L_SW__02") (unit 1) (value "L02 (C)") (footprint "burp_fart_keyswitches:Kailh_socket_MX_pads_flipped")
     )
     (path "/414fff57-7acf-4947-b712-fb535da1b8a4"
-      (reference "L_SW__3") (unit 1) (value "L03 (V)") (footprint "burp_fart_keyswitches:Kailh_socket_MX_pads_flipped")
+      (reference "L_SW__03") (unit 1) (value "L03 (V)") (footprint "burp_fart_keyswitches:Kailh_socket_MX_pads_flipped")
     )
     (path "/39b5118a-c07c-4df9-8796-01c96b1b183d"
-      (reference "L_SW__4") (unit 1) (value "L04 (B)") (footprint "burp_fart_keyswitches:Kailh_socket_MX_pads_flipped")
+      (reference "L_SW__04") (unit 1) (value "L04 (B)") (footprint "burp_fart_keyswitches:Kailh_socket_MX_pads_flipped")
     )
     (path "/7643cf93-d52d-4ac2-9b82-40915b8c98fa"
